File: ThumbsUp.kicad_pcb (KiCad board)
At the start: 2 copper layers, 251.1 x 336.1 mm, 120 parts, among them J1 Conn_01x04_Male, J10 Raiser_Male, J11 Raiser_Female, J12 Raiser_Male, J13 Raiser_Female, J14 Raiser_Male, J15 Raiser_Female, J16 Raiser_Male, J17 Raiser_Female, J18 Raiser_Male, J19 52559-1233, J2 Conn_01x04_Male, J20 Conn_01x04_Female, J21 Conn_01x04_Female, J22 Conn_01x04_Female, J23 Conn_01x04_Female, J24 Conn_01x04_Male, J25 Conn_01x04_Male, J26 Conn_01x04_Male, J27 Conn_01x04_Male, J28 Conn_01x04_Female, J29 Conn_01x04_Female, J3 Conn_01x04_Female, J30 Conn_01x04_Female, J31 Conn_01x04_Female, J4 Conn_01x04_Male, J5 Conn_01x04_Female, J6 Conn_01x04_Male, J7 Conn_01x04_Male, J8 Conn_01x04_Male, J9 Raiser_Female, U1 ProMicro

Commit message: WIP
Parts:
- added SW1: SW_Push, random-keyboard-parts:SKQG-1155865, F.Cu at (93.0, 238.0)
- U1: moved to F.Cu
- moved U1 28.5 mm to (147.1, 184.7)
Connections:
- U1 pad 1: Net-(U1-Pad1) -> ROW0
- U1 pad 10: Net-(U1-Pad10) -> COL4
- U1 pad 11: Net-(U1-Pad11) -> COL3
- U1 pad 12: Net-(U1-Pad12) -> COL2
- U1 pad 13: Net-(U1-Pad13) -> COL1
- U1 pad 14: Net-(U1-Pad14) -> COL0
- U1 pad 15: Net-(U1-Pad15) -> COL6
- U1 pad 16: Net-(U1-Pad16) -> COLB
- U1 pad 17: Net-(U1-Pad17) -> COLA
- U1 pad 18: Net-(U1-Pad18) -> COL9
- U1 pad 19: Net-(U1-Pad19) -> COL8
- U1 pad 2: Net-(U1-Pad2) -> ROW1
- U1 pad 20: Net-(U1-Pad20) -> COL7
- U1 pad 21: Net-(U1-Pad21) -> VCC
- U1 pad 22: Net-(U1-Pad22) -> RST
- U1 pad 23: Net-(U1-Pad23) -> GND
- U1 pad 5: Net-(U1-Pad5) -> SDA
- U1 pad 6: Net-(U1-Pad6) -> SCL
- U1 pad 7: Net-(U1-Pad7) -> ROW2
- U1 pad 8: Net-(U1-Pad8) -> ROW3
- U1 pad 9: Net-(U1-Pad9) -> COL5
Routing:
- net GND: track 253.8 -> 0.00 mm, vias 7 -> 0
- net VCC: track 154.3 -> 0.00 mm, vias 5 -> 0
- net ROW2: track 125.7 -> 27.0 mm, vias 2 -> 0
- net ROW3: track 142.9 -> 45.2 mm, vias 2 -> 0
- net COL2: track 137.4 -> 66.9 mm, vias 4 -> 1
- net COL6: track 182.5 -> 113.0 mm, vias 5 -> 3
- net ROW0: track 96.1 -> 29.3 mm, vias 4 -> 2
- net COL7: track 198.5 -> 133.4 mm, vias 4 -> 2
- net COLB: track 125.0 -> 63.0 mm, vias 1 -> 0
- net COLA: track 122.1 -> 63.0 mm, vias 1 -> 0
- net COL9: track 138.2 -> 80.4 mm, vias 1 -> 0
- net COL8: track 152.0 -> 96.4 mm, vias 1 -> 0
- net COL3: track 130.5 -> 77.5 mm, vias 1 -> 0
- net ROW1: track 73.6 -> 24.5 mm, vias 2 -> 0
- net COL0: track 101.8 -> 56.6 mm, vias 1 -> 0
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
Commit message: Routed the second layer, prepared for plotting
Parts:
- added G***: LOGO, Silkscreens:Crowfeet75, F.Cu at (144.3, 162.4)
- added G***: LOGO, Silkscreens:Crowfeet75, B.Cu at (146.4, 317.2)
- SW1: moved to B.Cu
- moved SW1 75.1 mm to (167.3, 227.4)
- moved D34 40.0 mm to (150.8, 211.3)
- moved D23 40.0 mm to (150.8, 208.9)
- moved D26 40.0 mm to (150.8, 220.9)
- moved D31 40.0 mm to (150.8, 218.5)
- moved D32 40.0 mm to (150.8, 216.1)
- moved D33 40.0 mm to (150.8, 213.7)
- moved D1 40.0 mm to (142.5, 218.5)
- moved D15 40.0 mm to (142.5, 220.9)
- moved D2 40.0 mm to (142.5, 216.1)
- moved D20 40.0 mm to (142.5, 209.0)
- moved D3 40.0 mm to (142.5, 213.7)
- moved D4 40.0 mm to (142.5, 211.3)
- moved D24 24.9 mm to (159.0, 208.9)
- moved D27 24.9 mm to (159.0, 220.9)
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Routing:
- net ROW2: track 27.0 -> 136.3 mm, vias 0 -> 2
- net GND: track 0.00 -> 107.4 mm
- net ROW3: track 45.2 -> 151.4 mm, vias 0 -> 2
- net SDA: track 6.89 -> 79.4 mm
- net VCC: track 0.00 -> 71.8 mm
- net RST: track 0.00 -> 71.1 mm, vias 0 -> 1
- net ROW1: track 24.5 -> 93.9 mm, vias 0 -> 1
- net SCL: track 9.95 -> 78.3 mm
- net COL0: track 56.6 -> 124.5 mm, vias 0 -> 1
- net COL1: track 56.8 -> 122.7 mm, vias 0 -> 1
- net Net-(D23-Pad2): track 24.0 -> 85.4 mm, vias 0 -> 1
- net COL8: track 96.4 -> 155.4 mm, vias 0 -> 1
- net COL9: track 80.4 -> 135.9 mm, vias 0 -> 1
- net COLA: track 63.0 -> 117.1 mm, vias 0 -> 1
- net COLB: track 63.0 -> 115.7 mm, vias 0 -> 1
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Other:
- outline, holes or cut-outs redrawn
- board text added: "Place ProMicro face to the plate."
- board text added: "QMK: #define MATRIX_ROW_PINS {D3,D2,D4,C6} #define MATRIX_COL_PINS {B2, B6, B5, B4,E6, D7, B3, F4, F5,F6, F7, B1} #define DIODE_DIRECTION COL2ROW"
- board text added: "RESET"
- board text added: "|<"

Commit message: Added power connector, pullup resistors for the trackpad, made the promicro holes bigger to fit the sockets.
Parts:
- removed the G*** at (144.3, 162.4)
- removed the G*** at (146.4, 317.2)
- added G***: LOGO, Silkscreens:Crowfeet75, F.Cu at (145.9, 197.2)
- added J32: Battery, Connector_PinHeader_2.54mm:PinHeader_1x02_P2.54mm_Vertical, B.Cu at (148.3, 204.9)
- added POWER: SW_DIP_x01, 1825232-1:18252321, F.Cu at (127.7, 227.8)
- added R1: 5.1K, Resistor_SMD:R_0805_2012Metric, B.Cu at (174.2, 227.6)
- added R2: 5.1K, Resistor_SMD:R_0805_2012Metric, B.Cu at (174.2, 225.6)
- moved SW1 6.55 mm to (160.8, 226.8)
Routing:
- net GND: track 107.4 -> 148.5 mm
- net Net-(J32-Pad2): track 0.00 -> 37.1 mm
- net COL6: track 148.8 -> 170.8 mm
- net VCC: track 71.8 -> 85.9 mm, vias 0 -> 1
- net RST: track 71.1 -> 64.2 mm
- net SCL: track 78.3 -> 84.7 mm
- net SDA: track 79.4 -> 84.2 mm
- net ROW1: track 93.9 -> 89.1 mm
- net ROW0: track 71.4 -> 74.0 mm
- net COL3: track 128.1 -> 127.2 mm
- net COL1: track 122.7 -> 121.8 mm
- net COL2: track 117.1 -> 116.3 mm
- net ROW3: track 151.4 -> 150.6 mm
- net COL0: track 124.5 -> 123.9 mm
Other:
- board text added: "Battery +RED HERE"
- board text added: "QMK: #define MATRIX_ROW_PINS {D3, D2, D4, C6} #define MATRIX_COL_PINS {B2, B6, B5, B4, E6, D7, B3, F4, F5, F6, F7, B1} #define DIODE_DIRECTION COL2ROW"
- board text removed: "QMK: #define MATRIX_ROW_PINS {D3,D2,D4,C6} #define MATRIX_COL_PINS {B2, B6, B5, B4,E6, D7, B3, F4, F5,F6, F7, B1} #define DIODE_DIRECTION COL2ROW"

Commit message: Regenerated Gerber for the middle layer.
Other:
- board text added: "Thumbs Up! by Sasha Karmanov October 28, 2022 https://github.com/ak66666/ ThumbsUpUnsplitV2ProMicro"
- board text removed: "Thumbs Up! by Sasha Karmanov October 28, 2022 https://github.com/ak66666/ThumbsUpUnsplitV2"
Changed lines of the file:
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@@
   (gr_line (start 153.416 169.418) (end 140.208 169.418) (layer Edge.Cuts) (width 0.05))
   (gr_circle (center 150.2 86.45) (end 152 66.4) (layer F.SilkS) (width 0.12))
-  (gr_text "Thumbs Up! by Sasha Karmanov\nOctober 28, 2022\nhttps://github.com/ak66666/ThumbsUpUnsplitV2" (at 146.15 360.3) (layer F.SilkS)
-    (effects (font (size 1 1) (thickness 0.15)))
+  (gr_text "Thumbs Up! by Sasha Karmanov\nOctober 28, 2022\nhttps://github.com/ak66666/\nThumbsUpUnsplitV2ProMicro" (at 110.3 216.37) (layer B.SilkS)
+    (effects (font (size 1 1) (thickness 0.15)) (justify mirror))
   )
   (gr_line (start 242.2 184.75) (end 226.45 190.75) (layer F.SilkS) (width 0.12))
